File: schematics/st_pat.kicad_sch (KiCad schematic)
At the start: 15 parts, among them J4 BATTERY, SW1 SW_PWR, SW2 BTN_RST, SW3 BTN, SW4 BTN, SW5 BTN, U1 GPS_Breakout_746, U2 FEATHER_M0_BASIC_PROTO, U3 LIS2MDL_ADAFRUIT, U4 Sharp_Display_4694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

Commit message: update display and telemetry breakout footprints
Connections:
- net +3V3: now also U3.2 (3v3); no longer U3.1 (VCC)
Changed lines of the file:
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@@
   (no_connect (at 106.68 59.69))
   (no_connect (at 199.39 116.84))
+  (no_connect (at 120.65 115.57))
   (no_connect (at 243.84 48.26))
   (no_connect (at 106.68 52.07))
   (no_connect (at 243.84 55.88))
-  (no_connect (at 120.65 119.38))
   (no_connect (at 48.26 52.07))
   (no_connect (at 167.64 52.07))
@@
   )
   (wire (pts (xy 184.15 134.62) (xy 199.39 134.62))
-    (stroke (width 0) (type default) (color 0 0 0 0))
-  )
-  (wire (pts (xy 113.03 115.57) (xy 120.65 115.57))
     (stroke (width 0) (type default) (color 0 0 0 0))
   )
@@
     (stroke (width 0) (type default) (color 0 0 0 0))
   )
+  (wire (pts (xy 120.65 119.38) (xy 113.03 119.38))
+    (stroke (width 0) (type default) (color 0 0 0 0))
+  )
   (wire (pts (xy 251.46 116.84) (xy 251.46 127))
     (stroke (width 0) (type default) (color 0 0 0 0))
@@
     (stroke (width 0) (type default) (color 0 0 0 0))
   )
+  (wire (pts (xy 113.03 119.38) (xy 113.03 115.57))
+    (stroke (width 0) (type default) (color 0 0 0 0))
+  )

Commit message: fix sch review issues
Connections:
- net GPS_PPS_D12 is gone; now on net GPS_PPS_D20: U1.1 (PPS)
- net +3V3: now also U3.1 (VCC); no longer U3.2 (3v3)
- net GPS_PPS_D20: now reaches U2.P2_12 (PA22/EINT/I2C/SDA)
- net GPS_PPS_D9: no longer names the net of U2.P2_8 (PA07/EINT/I2SD0)
Changed lines of the file:
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@@
   (junction (at 173.99 46.99) (diameter 0) (color 0 0 0 0)
   )
+  (no_connect (at 120.65 119.38))
   (no_connect (at 189.23 119.38))
   (no_connect (at 66.04 52.07))
   (no_connect (at 106.68 59.69))
   (no_connect (at 199.39 116.84))
-  (no_connect (at 120.65 115.57))
   (no_connect (at 243.84 48.26))
   (no_connect (at 106.68 52.07))
@@
   (no_connect (at 66.04 55.88))
   (no_connect (at 106.68 57.15))
-  (no_connect (at 167.64 85.09))
+  (no_connect (at 167.64 74.93))
   (no_connect (at 219.71 52.07))
   (no_connect (at 199.39 127))
@@
     (stroke (width 0) (type default) (color 0 0 0 0))
   )
-  (wire (pts (xy 120.65 119.38) (xy 113.03 119.38))
-    (stroke (width 0) (type default) (color 0 0 0 0))
-  )
   (wire (pts (xy 251.46 116.84) (xy 251.46 127))
     (stroke (width 0) (type default) (color 0 0 0 0))
@@
     (stroke (width 0) (type default) (color 0 0 0 0))
   )
-  (wire (pts (xy 113.03 119.38) (xy 113.03 115.57))
+  (wire (pts (xy 113.03 115.57) (xy 120.65 115.57))
     (stroke (width 0) (type default) (color 0 0 0 0))
   )
-  (text "P2_8 (D9) IS BATTERY MONITOR, DO NOT USE" (at 176.53 85.09 0)
+  (text "P2_8 (D9) IS BATTERY MONITOR, DO NOT USE" (at 172.72 88.9 0)
     (effects (font (size 1.27 1.27)) (justify left bottom))
   )
@@
     (effects (font (size 1.27 1.27)) (justify right bottom))
   )
-  (label "GPS_PPS_D12" (at 48.26 48.26 180)
+  (label "GPS_PPS_D20" (at 48.26 48.26 180)
     (effects (font (size 1.27 1.27)) (justify right bottom))
   )
@@
     (effects (font (size 1.27 1.27)) (justify right bottom))
   )
-  (label "GPS_PPS_D9" (at 167.64 74.93 0)
+  (label "GPS_PPS_D20" (at 167.64 85.09 0)
     (effects (font (size 1.27 1.27)) (justify left bottom))
   )

Commit message: fix typo in schematic and remove calibration test code
Connections:
- net TELE_RX_D12 renamed TELE_RX_D11
- net TELE_TX_D11 renamed TELE_TX_D12
Changed lines of the file:
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@@
     (effects (font (size 1.27 1.27)) (justify left bottom))
   )
-  (label "TELE_RX_D12" (at 53.34 124.46 180)
+  (label "TELE_RX_D11" (at 53.34 124.46 180)
     (effects (font (size 1.27 1.27)) (justify right bottom))
   )
@@
     (effects (font (size 1.27 1.27)) (justify right bottom))
   )
-  (label "TELE_RX_D12" (at 167.64 69.85 0)
+  (label "TELE_RX_D11" (at 167.64 69.85 0)
     (effects (font (size 1.27 1.27)) (justify left bottom))
   )
@@
     (effects (font (size 1.27 1.27)) (justify left bottom))
   )
-  (label "TELE_TX_D11" (at 167.64 67.31 0)
+  (label "TELE_TX_D12" (at 167.64 67.31 0)
     (effects (font (size 1.27 1.27)) (justify left bottom))
   )
@@
     (effects (font (size 1.27 1.27)) (justify right bottom))
   )
-  (label "TELE_TX_D11" (at 53.34 128.27 180)
+  (label "TELE_TX_D12" (at 53.34 128.27 180)
     (effects (font (size 1.27 1.27)) (justify right bottom))
   )
